File: Hardware/PCB/Transmisor/Telemetria.sch (EAGLE design)
At the start: 11 parts, among them X3 JST-XH-05-PIN-LONG-PAD

Commit message: fix(transmissor): transmisson pcb updated
Parts:
- LORA_STATUS_LED: value (none) -> BLUE
- MCP_STATUS_LED: value (none) -> RED
- R1: value (none) -> 150
- R10: value (none) -> 100
- X4: value (none) -> DV9
Connections:
- net LORA_NSS: now also B1.D8; no longer B1.*D10
- net MCP_CS: now also B1.*D10; no longer B1.D8
Changed lines of the file:
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@@
 <parts>
 <part name="B1" library="SparkFun-Boards" library_urn="urn:adsk.eagle:library:509" deviceset="ARDUINO_UNO_R3_SHIELD_ICSP" device="-NO_LABELS" package3d_urn="urn:adsk.eagle:package:37336/1"/>
-<part name="R10" library="resistor" library_urn="urn:adsk.eagle:library:348" deviceset="R-US_" device="M0805" package3d_urn="urn:adsk.eagle:package:26079/1"/>
-<part name="LORA_STATUS_LED" library="led" library_urn="urn:adsk.eagle:library:259" deviceset="LED" device="CHIP-LED0805" package3d_urn="urn:adsk.eagle:package:15818/1"/>
+<part name="R10" library="resistor" library_urn="urn:adsk.eagle:library:348" deviceset="R-US_" device="M0805" package3d_urn="urn:adsk.eagle:package:26079/1" value="100"/>
+<part name="LORA_STATUS_LED" library="led" library_urn="urn:adsk.eagle:library:259" deviceset="LED" device="CHIP-LED0805" package3d_urn="urn:adsk.eagle:package:15818/1" value="BLUE"/>
 <part name="GND1" library="supply1" library_urn="urn:adsk.eagle:library:371" deviceset="GND" device=""/>
 <part name="GND2" library="supply1" library_urn="urn:adsk.eagle:library:371" deviceset="GND" device=""/>
 <part name="GND3" library="supply1" library_urn="urn:adsk.eagle:library:371" deviceset="GND" device=""/>
 <part name="GND4" library="supply1" library_urn="urn:adsk.eagle:library:371" deviceset="GND" device=""/>
-<part name="R1" library="resistor" library_urn="urn:adsk.eagle:library:348" deviceset="R-US_" device="M0805" package3d_urn="urn:adsk.eagle:package:26079/1"/>
-<part name="MCP_STATUS_LED" library="led" library_urn="urn:adsk.eagle:library:259" deviceset="LED" device="CHIP-LED0805" package3d_urn="urn:adsk.eagle:package:15818/1"/>
+<part name="R1" library="resistor" library_urn="urn:adsk.eagle:library:348" deviceset="R-US_" device="M0805" package3d_urn="urn:adsk.eagle:package:26079/1" value="150"/>
+<part name="MCP_STATUS_LED" library="led" library_urn="urn:adsk.eagle:library:259" deviceset="LED" device="CHIP-LED0805" package3d_urn="urn:adsk.eagle:package:15818/1" value="RED"/>
 <part name="GND5" library="supply1" library_urn="urn:adsk.eagle:library:371" deviceset="GND" device=""/>
 <part name="P+1" library="supply1" library_urn="urn:adsk.eagle:library:371" deviceset="+5V" device=""/>
@@
 <part name="SPI" library="Rembrandt Electronics - JST XH Connectors v1-0" deviceset="JST-XH-05-PIN" device="-LONG-PAD"/>
 <part name="X3" library="Rembrandt Electronics - JST XH Connectors v1-0" deviceset="JST-XH-05-PIN" device="-LONG-PAD"/>
-<part name="X4" library="con-subd" library_urn="urn:adsk.eagle:library:189" deviceset="F09" device="H" package3d_urn="urn:adsk.eagle:package:10276/1"/>
+<part name="X4" library="con-subd" library_urn="urn:adsk.eagle:library:189" deviceset="F09" device="H" package3d_urn="urn:adsk.eagle:package:10276/1" value="DV9"/>
 <part name="GND8" library="supply1" library_urn="urn:adsk.eagle:library:371" deviceset="GND" device=""/>
 <part name="MCP2515" library="EL_POTENCIA_LIBRERIA_VES2018" deviceset="MCP2515" device=""/>
@@
 <instance part="R10" gate="G$1" x="13.97" y="30.48" smashed="yes">
 <attribute name="NAME" x="11.43" y="26.8986" size="1.778" layer="95"/>
-<attribute name="VALUE" x="10.16" y="27.178" size="1.778" layer="96"/>
+<attribute name="VALUE" x="16.764" y="26.924" size="1.778" layer="96"/>
 </instance>
 <instance part="LORA_STATUS_LED" gate="G$1" x="-2.54" y="30.48" smashed="yes" rot="R90">
 <attribute name="NAME" x="-3.302" y="33.274" size="1.778" layer="95"/>
-<attribute name="VALUE" x="2.032" y="36.195" size="1.778" layer="96" rot="R180"/>
 </instance>
 <instance part="GND1" gate="1" x="-66.04" y="-2.54" smashed="yes" rot="R270">
@@
 <instance part="R1" gate="G$1" x="13.97" y="20.32" smashed="yes">
 <attribute name="NAME" x="11.43" y="16.7386" size="1.778" layer="95"/>
-<attribute name="VALUE" x="10.16" y="17.018" size="1.778" layer="96"/>
+<attribute name="VALUE" x="15.748" y="16.764" size="1.778" layer="96"/>
 </instance>
 <instance part="MCP_STATUS_LED" gate="G$1" x="-2.54" y="20.32" smashed="yes" rot="R90">
 <attribute name="NAME" x="-3.302" y="23.114" size="1.778" layer="95"/>
-<attribute name="VALUE" x="2.032" y="26.035" size="1.778" layer="96" rot="R180"/>
+<attribute name="VALUE" x="25.146" y="25.019" size="1.778" layer="96" rot="R180"/>
 </instance>
 <instance part="GND5" gate="1" x="29.21" y="20.32" smashed="yes" rot="R90">
@@
 <net name="MCP_CS" class="0">
 <segment>
-<pinref part="B1" gate="G$1" pin="D8"/>
-<wire x1="-29.21" y1="7.62" x2="-25.4" y2="7.62" width="0.1524" layer="91"/>
-<label x="-25.4" y="7.62" size="1.778" layer="95" xref="yes"/>
-</segment>
-<segment>
 <pinref part="MCP2515" gate="G$1" pin="CS"/>
 <wire x1="53.34" y1="-35.56" x2="55.88" y2="-35.56" width="0.1524" layer="91"/>
 <label x="55.88" y="-35.56" size="1.778" layer="95" xref="yes"/>
+</segment>
+<segment>
+<pinref part="B1" gate="G$1" pin="*D10"/>
+<wire x1="-29.21" y1="2.54" x2="-27.94" y2="2.54" width="0.1524" layer="91"/>
+<label x="-27.94" y="2.54" size="1.778" layer="95" xref="yes"/>
 </segment>
 </net>
@@
 <net name="LORA_NSS" class="0">
 <segment>
-<pinref part="B1" gate="G$1" pin="*D10"/>
-<wire x1="-29.21" y1="2.54" x2="-27.94" y2="2.54" width="0.1524" layer="91"/>
-<label x="-27.94" y="2.54" size="1.778" layer="95" xref="yes"/>
-</segment>
-<segment>
 <pinref part="LORA_RA-02" gate="G$1" pin="NSS"/>
 <wire x1="58.42" y1="2.54" x2="60.96" y2="2.54" width="0.1524" layer="91"/>
 <label x="60.96" y="2.54" size="1.778" layer="95" xref="yes"/>
 </segment>
-</net>
+<segment>
+<pinref part="B1" gate="G$1" pin="D8"/>
+<wire x1="-29.21" y1="7.62" x2="-27.94" y2="7.62" width="0.1524" layer="91"/>
+<label x="-27.94" y="7.62" size="1.778" layer="95" xref="yes"/>
+</segment>
+</net>
