File: Hardware/PCB/Coordinator/Coordinator.sch (EAGLE design)
At the start: 9 parts, among them IC1 TLV2217-33KCSE3, X1 JST-XH-02-PIN-LONG-PAD

Commit message: commit after race
Parts:
- renumbered IC1 to TVL2217-33, LED1 to 0805GREEN, LED2 to 0805BLUE, U$1 to LORA
Connections:
- net N$3 renamed 3.3V
- net N$7 renamed IRQ
- net N$8 renamed LORA_RST
- removed net N$1: B1.GND@2, TVL2217-33.GND, X1-1.S
- removed net N$2: B1.VCC, TVL2217-33.INPUT, X1-2.S
- removed net N$4: B1.GND, JP1.1
- net GND: now also JP1.1, TVL2217-33.GND, X1-1.S
- net VCC: now also B1.VCC, TVL2217-33.INPUT, X1-2.S
